Commit message: fix: TD3 training bugs, Gazebo wiring, sensor model and lbt_control packaging
- td3: critic used .weight.data for layer_2/5, so those weights never trained
- td3: target-policy noise was written in-place over the sampled batch actions
- environment: portable world path, real world name (maze_world), clip inf ranges
- spawn_maze: bridge control/set_pose services; spawn inside the maze
- lidar xacro: gazebo reference pointed at a non-existent link (no scans);
  sensors now sit on their mesh face and point outward
- lbt_control: add console_script and launch install, fix xacro path and
  ParameterValue kwarg, use URDF wheel joint names, declare runtime deps
- train/eval: local imports so the scripts run directly

Co-Authored-By: Claude Opus 5.5 <noreply@anthropic.com>
Claude-Session: https://claude.ai/code/session_01Rf1kKiTUEpSBhFeLv7FvGN

File: ros_space/lbrtia/src/lbt_description/urdf/rbt.urdf.xacro (robot description, xacro)
@@ -125,7 +125,9 @@
   </joint>
   <!-- ===== Macros de sensores (padres = los enlaces creados) ===== -->
-  <xacro:hc_sr04_lidar prefix="hc_sr04_left"   parent="hc_left"   topic="scan_left"   xyz="0 0 0" rpy="0 0 0"/>
-  <xacro:hc_sr04_lidar prefix="hc_sr04_center" parent="hc_front" topic="scan_center" xyz="0 0 0" rpy="0 0 0"/>
-  <xacro:hc_sr04_lidar prefix="hc_sr04_right"  parent="hc_right" topic="scan_right"  xyz="0 0 0" rpy="0 0 0"/>
+  <!-- xyz/rpy en el marco de cada malla hc_*: cara exterior de la malla, apuntando hacia afuera
+       (hc_c -> +X del robot, hc_l -> -Y, hc_r -> +Y) -->
+  <xacro:hc_sr04_lidar prefix="hc_sr04_left"   parent="hc_left"   topic="scan_left"   xyz="0.0475 0 0.0105"  rpy="0 0 0"/>
+  <xacro:hc_sr04_lidar prefix="hc_sr04_center" parent="hc_front" topic="scan_center" xyz="0 0.0403 0.0105"  rpy="0 0 1.5708"/>
+  <xacro:hc_sr04_lidar prefix="hc_sr04_right"  parent="hc_right" topic="scan_right"  xyz="-0.0484 0 0.0105" rpy="0 0 3.14159"/>
   <!-- ===== Rueda Izquierda ===== -->
   <link name="rueda_izquierda">

File: ros_space/lbrtia/src/lbt_description/urdf/sensors/hc_sr04_lidar.xacro (robot description, xacro)
@@ -2,9 +2,9 @@
 <robot xmlns:xacro="http://ros.org/wiki/xacro">
   <xacro:macro name="hc_sr04_lidar" params="prefix parent topic xyz rpy">
-    <link name="${prefix}">
+    <link name="${prefix}_link">
     </link>
     <joint name="${prefix}_joint" type="fixed">
       <parent link="${parent}"/>
-      <child link="${prefix}"/>
+      <child link="${prefix}_link"/>
       <origin xyz="${xyz}" rpy="${rpy}"/>
     </joint>

Commit message: feat: lightweight RViz simulation (lbt_sim) and pending fixes
- lbt_sim: 2D kinematic simulator (cmd_vel -> pose, raycast HC-SR04 scans
  against maze.world walls, /odom, /tf, /joint_states, wall markers) that
  serves the same control/set_pose services lbt_ai uses with Gazebo
- rviz_sim.launch.py + sim.rviz; train/eval default to it
- URDF: Gazebo diff-drive, ground-truth odometry and joint-state plugins;
  right wheel axis flipped so both wheels drive forward; world loads IMU system
- environment: COLLISION_DIST 0.15, spawn margin 0.25, reuse parse_maze_walls
- lbt_control: odom child frame base_footprint (base already had a parent)
- remove dead legacy code (lbrintia/, lbt_ai/train.py) and untrack install/, log/

Co-Authored-By: Claude Opus 5.5 <noreply@anthropic.com>
Claude-Session: https://claude.ai/code/session_01Rf1kKiTUEpSBhFeLv7FvGN

File: ros_space/lbrtia/src/lbt_description/urdf/rbt.urdf.xacro (robot description, xacro)
@@ -187,8 +187,36 @@
     <parent link="base"/>
     <child link="rueda_derecha"/>
-    <axis xyz="0 0 1"/>
+    <!-- invertido para que, como en rueda_izquierda, girar en positivo haga avanzar el robot -->
+    <axis xyz="0 0 -1"/>
     <limit effort="10" velocity="10"/>
   </joint>
   <!-- ===== Sensor IMU (macro) ===== -->
   <xacro:imu_sensor prefix="imu" parent="base" topic="imu" xyz="0 0 0.01" rpy="0 0 0"/>
+  <!-- ===== Plugins de Gazebo (spawn_maze.launch.py; la simulación en RViz usa lbt_sim) ===== -->
+  <gazebo>
+    <plugin filename="gz-sim-diff-drive-system" name="gz::sim::systems::DiffDrive">
+      <!-- rueda_derecha está en +Y (izquierda según ROS) y rueda_izquierda en -Y -->
+      <left_joint>joint_rueda_derecha</left_joint>
+      <right_joint>joint_rueda_izquierda</right_joint>
+      <wheel_separation>0.125</wheel_separation>
+      <wheel_radius>0.033</wheel_radius>
+      <topic>/cmd_vel</topic>
+      <!-- odometría de ruedas fuera de /odom: no sigue los teletransportes del reset de lbt_ai -->
+      <odom_topic>/odom_wheels</odom_topic>
+      <tf_topic>/tf_wheels</tf_topic>
+      <frame_id>odom</frame_id>
+      <child_frame_id>base_footprint</child_frame_id>
+    </plugin>
+    <plugin filename="gz-sim-odometry-publisher-system" name="gz::sim::systems::OdometryPublisher">
+      <odom_frame>odom</odom_frame>
+      <robot_base_frame>base_footprint</robot_base_frame>
+      <odom_topic>/odom</odom_topic>
+      <tf_topic>/tf</tf_topic>
+      <dimensions>2</dimensions>
+      <odom_publish_frequency>50</odom_publish_frequency>
+    </plugin>
+    <plugin filename="gz-sim-joint-state-publisher-system" name="gz::sim::systems::JointStatePublisher">
+      <topic>/joint_states</topic>
+    </plugin>
+  </gazebo>
 </robot>
